File: KiCad/IrController.sch (KiCad schematic (older format))
At the start: 7 parts, among them J11 IrJack, J12 ICSP, U1 PIC16F15325

Commit message: Added KiCad footprints + fixed library references in schematic
Parts:
- J11: symbol IrOutlet-rescue:AudioJack3-IrOutlet-IrOutlet-rescue-IrOutlet-rescue -> IrOutlet:AudioJack3
- U1: symbol IrOutlet-rescue:PIC16F15325-IrOutlet-IrOutlet-rescue-IrOutlet-rescue -> IrOutlet:PIC16F15325
Changed lines of the file:
@@
 Connection ~ 3250 3800
 $Comp
-L IrOutlet-rescue:PIC16F15325-IrOutlet-IrOutlet-rescue-IrOutlet-rescue U1
+L IrOutlet:PIC16F15325 U1
 U 1 1 5FA43535
 P 4150 4200
@@
 $EndComp
 $Comp
-L IrOutlet-rescue:AudioJack3-IrOutlet-IrOutlet-rescue-IrOutlet-rescue J11
+L IrOutlet:AudioJack3 J11
 U 1 1 5FA65205
 P 5100 6900
