File: KiCad/IrOutlet.kicad_pcb (KiCad board)
At the start: 2 copper layers, 250 x 100 mm, 66 parts, among them J1 OUT, J10 5V, J11 IR Jack, J12 ICSP, J2 OUT, J3 OUT, J4 OUT, J5 OUT, J6 OUT, J7 OUT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

Commit message: Added KiCad footprints + fixed library references in schematic
Parts:
- C2: value 47uF -> 100uF
- D1: value 1N4007 -> 1N5819
- J11: value IR Jack -> IrJack
Changed lines of the file:
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@@
       (effects (font (size 1 1) (thickness 0.15)))
     )
-    (fp_text value 47uF (at 1.25 4.4) (layer F.Fab) hide
+    (fp_text value 100uF (at 1.25 4.4) (layer F.Fab) hide
       (effects (font (size 1 1) (thickness 0.15)))
     )
@@
       (effects (font (size 1 1) (thickness 0.15)))
     )
-    (fp_text value 1N4007 (at 5.08 2.47) (layer F.Fab) hide
+    (fp_text value 1N5819 (at 5.08 2.47) (layer F.Fab) hide
       (effects (font (size 1 1) (thickness 0.15)))
     )
@@
       (effects (font (size 1 1) (thickness 0.15)))
     )
-    (fp_text value "IR Jack" (at 0 7.41) (layer F.Fab) hide
-      (effects (font (size 1 1) (thickness 0.15)))
-    )
+    (fp_text value IrJack (at 0 7.41) (layer F.Fab) hide
+      (effects (font (size 1 1) (thickness 0.15)))
+    )
